File: hardware/hardware/hardware.kicad_pcb (KiCad board)
At the start: 2 copper layers, 17 parts, among them IC1 TM1637, J1 SENSOR, J2 POWER, J3 ISP, U1 ATtiny45V, U2 LM78M05

Commit message: pcb
Parts:
- removed C4: 10uF, Capacitor_SMD:CP_Elec_6.3x5.8
- removed J3: ISP, Connector_PinHeader_2.54mm:PinHeader_2x03_P2.54mm_Vertical
- removed U2: LM78M05, Package_TO_SOT_SMD:TO-252-2
- added C2: 10uF, Capacitor_SMD:C_0805_2012Metric, B.Cu at (144.4, 59.2)
- added U3: AMS1117-5.0, Package_TO_SOT_SMD:SOT-223-3_TabPin2, B.Cu at (149.5, 58.6)
- C1: footprint Capacitor_SMD:CP_Elec_6.3x5.8 -> Capacitor_SMD:C_0805_2012Metric
- D3: value 2841BS -> 5631BS; footprint 2841BS:2841BS -> 5631BS:5631BS
- IC1, U1: moved to B.Cu
- R1: moved to F.Cu
- moved R4 71.3 mm to (122.5, 50.9), turned to 180 degrees
- moved R3 70.3 mm to (122.5, 48.8), turned to 180 degrees
- moved U1 70.2 mm to (122.6, 57.3)
- moved D2 69.6 mm to (149.4, 50.6), turned to 180 degrees
- moved C1 69.5 mm to (144.4, 54.2), turned to -90 degrees
- moved IC1 68.1 mm to (135.9, 57.1)
- moved R2 65.0 mm to (119.4, 58.2)
- moved D1 62.4 mm to (119.4, 61.9), turned to 90 degrees
- moved D3 59.2 mm to (129.7, 64.6)
- moved J2 57.3 mm to (158.5, 50.7)
- moved C6 55.0 mm to (126.8, 56.3), turned to 0 degrees
- moved C5 49.0 mm to (126.8, 59.6), turned to 0 degrees
- moved J1 45.4 mm to (158.4, 57.7), turned to -90 degrees
- moved R1 35.9 mm to (155.5, 60.4), turned to 90 degrees
Connections:
- net /MISO renamed Net-(U1-PB1)
- net /MOSI renamed Net-(IC1-DIO)
- net /SCK renamed Net-(IC1-CLK)
- U1 pad 1: /RST -> unconnected-(U1-~{RESET}/PB5-Pad1)
Routing:
- net +5V: track 0.00 -> 60.0 mm, vias 0 -> 3
- net Net-(J1-Pin_2): track 0.00 -> 43.8 mm, vias 0 -> 1
- net Net-(IC1-DIO): track 0.00 -> 35.5 mm, vias 0 -> 4
- net Net-(D3-a): track 0.00 -> 28.2 mm
- net Net-(IC1-CLK): track 0.00 -> 26.7 mm
- net Net-(D3-f): track 0.00 -> 25.9 mm, vias 0 -> 1
- net Net-(D3-g): track 0.00 -> 21.2 mm, vias 0 -> 1
- net Net-(D3-b): track 0.00 -> 13.9 mm, vias 0 -> 1
- net Net-(D3-e): track 0.00 -> 13.8 mm, vias 0 -> 1
- net Net-(D2-A): track 0.00 -> 13.1 mm
- net +12V: track 0.00 -> 12.4 mm
- net /CA3: track 0.00 -> 12.3 mm, vias 0 -> 1
- net /CA1: track 0.00 -> 12.2 mm, vias 0 -> 1
- net Net-(D3-DPX): track 0.00 -> 9.34 mm, vias 0 -> 1
- net Net-(D3-d): track 0.00 -> 6.08 mm
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- added copper zone on B.Cu, net GND
- added copper zone on F.Cu, net GND
Other:
- board outline added: 45.2 x 20.1 mm
- board text added: "+"

Commit message: pcb
Routing:
- net Net-(IC1-DIO): track 35.5 -> 37.6 mm
- net /CA3: track 12.3 -> 13.6 mm
- net Net-(D3-g): track 21.2 -> 22.1 mm
Other:
- board size 45.2 x 20.1 mm -> 46.2 x 21.1 mm
- board text added: "GND"

Commit message: pcb
Parts:
- added REF**: MountingHole_2.2mm_M2, MountingHole:MountingHole_2.2mm_M2, F.Cu at (173.2, 103.2)
- added REF**: MountingHole_2.2mm_M2, MountingHole:MountingHole_2.2mm_M2, F.Cu at (173.2, 82.2)
- J1, J2: moved to F.Cu
- R1: moved to B.Cu
- moved J1 42.0 mm to (168.7, 98.4), turned to 90 degrees
- moved R1 40.0 mm to (159.8, 100.2), turned to 180 degrees
- moved J2 39.9 mm to (168.7, 89.2), turned to 90 degrees
- moved D1 37.2 mm to (129.6, 97.7)
- moved R4 37.2 mm to (132.7, 86.7)
- moved C1 37.2 mm to (154.6, 90.0)
- moved C2 37.2 mm to (154.6, 95.0)
- moved D3 37.2 mm to (139.9, 100.3)
- moved R2 37.2 mm to (129.6, 94.0)
- moved R3 37.2 mm to (132.7, 84.5)
- moved U1 37.2 mm to (132.8, 93.0)
- moved C6 37.2 mm to (136.9, 92.0)
- moved D2 37.2 mm to (159.6, 86.3)
- moved U2 37.2 mm to (146.1, 92.8)
- moved U3 37.2 mm to (159.7, 94.3)
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- renumbered IC1 to U2
Connections:
- J1 pad 1: +5V -> GND
- J1 pad 3: GND -> +5V
- J2 pad 1: Net-(D2-A) -> GND
- J2 pad 2: GND -> Net-(D2-A)
Routing:
- net Net-(J1-Pin_2): track 43.8 -> 46.0 mm, vias 1 -> 0
- net +5V: track 59.7 -> 60.5 mm, vias 3 -> 2
- net /CA1: track 12.0 -> 12.6 mm
