File: hardware/hardware/hardware.kicad_sch (KiCad schematic)
At the start: 11 parts, among them J1 POWER, J2 SENSOR, U1 ATtiny45V-10X, U2 LM78M05_TO252

Commit message: schematic
Parts:
- removed C3, C4: 330nF, Capacitor_SMD:C_0805_2012Metric, symbol Device:C_Small
- added C5, C6: 100pF, Capacitor_SMD:C_0805_2012Metric, symbol Device:C_Small
- added D3: 2841BS, 2841BS:2841BS, symbol 2841BS:2841BS
- added IC1: TM1637, TM1637__SOP_:SOIC127P1045X280-20N, symbol TM1637__SOP_:TM1637__SOP_
- added J3: ISP, Connector_PinHeader_2.54mm:PinHeader_2x03_P2.54mm_Vertical, symbol Connector:AVR-ISP-6
- added R2: 330, Resistor_SMD:R_0805_2012Metric, symbol Device:R
- added R3, R4: 10K, Resistor_SMD:R_0805_2012Metric, symbol Device:R
- C5: value 1000uF -> 10uF; footprint Capacitor_SMD:CP_Elec_10x10.5 -> Capacitor_SMD:CP_Elec_6.3x5.8
- C6: value 220uF -> 10uF; footprint Capacitor_SMD:CP_Elec_6.3x7.7 -> Capacitor_SMD:CP_Elec_6.3x5.8
- D1: value LED -> ERR; footprint (none) -> LED_SMD:LED_0805_2012Metric
- U1: value ATtiny45V-10X -> ATtiny45V
- U2: value LM78M05_TO252 -> LM78M05
Connections:
- net DQ is gone; now on an unnamed net: J2.2 (Pin_2), R2.1
- net +5V: now also U1.8 (VCC), IC1.16 (VDD), J3.2 (VCC), R3.1, R4.1
- net GND: now also D1.1 (K), U1.4 (GND), C5.2, C6.2, IC1.1 (GND), J3.6 (GND)
- net RST: now reaches U1.1 (~{RESET}/PB5)
- net RST: now also J3.5 (~{RST})
- net MOSI: now reaches U1.5 (AREF/PB0)
- net MOSI: now also C5.1, IC1.17 (DIO), J3.4 (MOSI), R3.2
- net MISO: now reaches U1.6 (PB1)
- net MISO: now also J3.1 (MISO), R2.1
- net SCK: now reaches U1.7 (PB2)
- net SCK: now also C6.1, IC1.18 (CLK), J3.3 (SCK), R4.2
- net at D1.2 (A): now also R2.2
- new net: D3.11 (a), IC1.2 (SEG1/KS1)
- new net: D3.7 (b), IC1.3 (SEG2/KS2)
- new net: D3.4 (c), IC1.4 (SEG3/KS3)
- new net: D3.2 (d), IC1.5 (SEG4/KS4)
- new net: D3.1 (e), IC1.6 (SEG5/KS5)
- new net: D3.10 (f), IC1.7 (SEG6/KS6)
- new net: D3.5 (g), IC1.8 (SEG7/KS7)
- new net: D3.3 (DPX), IC1.9 (SEG8/KS8)
- new net CA1: D3.12 (CA1), IC1.15 (GRID1)
- new net CA2: D3.9 (CA2), IC1.14 (GRID2)
- new net CA3: D3.8 (CA3), IC1.13 (GRID3)
- no-connect marks 0 -> 6
Other:
- moved on the sheet: C5, C6, D1, D4, J1, J2, R2, U1, U2

Commit message: pcb
Parts:
- removed C5, C6: 10uF, Capacitor_SMD:CP_Elec_6.3x5.8, symbol Device:C_Polarized
- removed D3: 2841BS, 2841BS:2841BS, symbol 2841BS:2841BS
- removed J3: ISP, Connector_PinHeader_2.54mm:PinHeader_2x03_P2.54mm_Vertical, symbol Connector:AVR-ISP-6
- removed U2: LM78M05, Package_TO_SOT_SMD:TO-252-2, symbol Regulator_Linear:LM78M05_TO252
- added C1, C2: 10uF, Capacitor_SMD:C_0805_2012Metric, symbol Device:C
- added D3: 5631BS, 5631BS:5631BS, symbol 5631BS:5631BS
- added U3: AMS1117-5.0, Package_TO_SOT_SMD:SOT-223-3_TabPin2, symbol Regulator_Linear:AMS1117-5.0
Connections:
- net +12V: now also C1.1, U3.3 (VI)
- net +5V: now also C2.1, U3.2 (VO)
- net CA1: now also D3.12 (CA1)
- net CA2: now also D3.9 (CA2)
- net CA3: now also D3.8 (CA3)
- net GND: now also C1.2, C2.2, U3.1 (GND)
- net at IC1.2 (SEG1/KS1): now also D3.11 (a)
- net at IC1.3 (SEG2/KS2): now also D3.7 (b)
- net at IC1.4 (SEG3/KS3): now also D3.4 (c)
- net at IC1.5 (SEG4/KS4): now also D3.2 (d)
- net at IC1.6 (SEG5/KS5): now also D3.1 (e)
- net at IC1.7 (SEG6/KS6): now also D3.10 (f)
- net at IC1.8 (SEG7/KS7): now also D3.5 (g)
- net at IC1.9 (SEG8/KS8): now also D3.3 (DPX)
- net MISO: no longer names the net of R2.1, U1.6 (PB1)
- net MOSI: no longer names the net of C5.1, IC1.17 (DIO), R3.2, U1.5 (AREF/PB0)
- net RST: no longer names the net of U1.1 (~{RESET}/PB5)
- net SCK: no longer names the net of C6.1, IC1.18 (CLK), R4.2, U1.7 (PB2)
- no-connect marks 6 -> 7

Commit message: pcb
Parts:
- renumbered IC1 to U2
Connections:
- net +5V: now also J2.3 (Pin_3); no longer J2.1 (Pin_1)
- net GND: now also J1.1 (Pin_1), J2.1 (Pin_1); no longer J1.2 (Pin_2), J2.3 (Pin_3)
- net at D4.2 (A): now also J1.2 (Pin_2); no longer J1.1 (Pin_1)
Other:
- moved on the sheet: J1
Changed lines of the file:
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@@
     (date "2023-08-08")
   )
+  (junction (at 163.83 39.37) (diameter 0) (color 0 0 0 0)
+  )
+  (junction (at 101.6 124.46) (diameter 0) (color 0 0 0 0)
+  )
+  (junction (at 142.24 95.25) (diameter 0) (color 0 0 0 0)
+  )
+  (junction (at 92.71 53.34) (diameter 0) (color 0 0 0 0)
+  )
+  (junction (at 77.47 39.37) (diameter 0) (color 0 0 0 0)
+  )
+  (junction (at 77.47 53.34) (diameter 0) (color 0 0 0 0)
+  )
+  (junction (at 144.78 63.5) (diameter 0) (color 0 0 0 0)
+  )
+  (junction (at 142.24 124.46) (diameter 0) (color 0 0 0 0)
+  )
   (junction (at 163.83 49.53) (diameter 0) (color 0 0 0 0)
-  )
-  (junction (at 163.83 39.37) (diameter 0) (color 0 0 0 0)
-  )
-  (junction (at 101.6 124.46) (diameter 0) (color 0 0 0 0)
-  )
-  (junction (at 142.24 95.25) (diameter 0) (color 0 0 0 0)
-  )
-  (junction (at 92.71 53.34) (diameter 0) (color 0 0 0 0)
-  )
-  (junction (at 77.47 39.37) (diameter 0) (color 0 0 0 0)
-  )
-  (junction (at 77.47 53.34) (diameter 0) (color 0 0 0 0)
-  )
-  (junction (at 144.78 63.5) (diameter 0) (color 0 0 0 0)
-  )
-  (junction (at 142.24 124.46) (diameter 0) (color 0 0 0 0)
   )
   (junction (at 147.32 100.33) (diameter 0) (color 0 0 0 0)
@@
     (stroke (width 0) (type default))
   )
+  (wire (pts (xy 50.8 41.91) (xy 53.34 41.91))
+    (stroke (width 0) (type default))
+  )
   (wire (pts (xy 147.32 100.33) (xy 163.83 100.33))
     (stroke (width 0) (type default))
@@
     (stroke (width 0) (type default))
   )
+  (wire (pts (xy 163.83 49.53) (xy 172.72 49.53))
+    (stroke (width 0) (type default))
+  )
   (wire (pts (xy 142.24 95.25) (xy 157.48 95.25))
     (stroke (width 0) (type default))
@@
     (stroke (width 0) (type default))
   )
+  (wire (pts (xy 163.83 49.53) (xy 163.83 53.34))
+    (stroke (width 0) (type default))
+  )
   (wire (pts (xy 199.39 100.33) (xy 212.09 100.33))
     (stroke (width 0) (type default))
@@
     (stroke (width 0) (type default))
   )
+  (wire (pts (xy 168.91 52.07) (xy 172.72 52.07))
+    (stroke (width 0) (type default))
+  )
   (wire (pts (xy 92.71 46.99) (xy 92.71 53.34))
     (stroke (width 0) (type default))
@@
     (stroke (width 0) (type default))
   )
-  (wire (pts (xy 50.8 41.91) (xy 53.34 41.91))
-    (stroke (width 0) (type default))
-  )
   (wire (pts (xy 21.59 39.37) (xy 21.59 43.18))
     (stroke (width 0) (type default))
@@
     (stroke (width 0) (type default))
   )
+  (wire (pts (xy 50.8 39.37) (xy 55.88 39.37))
+    (stroke (width 0) (type default))
+  )
   (wire (pts (xy 77.47 39.37) (xy 85.09 39.37))
     (stroke (width 0) (type default))
@@
     (stroke (width 0) (type default))
   )
-  (wire (pts (xy 50.8 39.37) (xy 55.88 39.37))
-    (stroke (width 0) (type default))
-  )
   (wire (pts (xy 142.24 95.25) (xy 142.24 110.49))
     (stroke (width 0) (type default))
@@
     (stroke (width 0) (type default))
   )
-  (wire (pts (xy 172.72 52.07) (xy 168.91 52.07))
-    (stroke (width 0) (type default))
-  )
   (wire (pts (xy 144.78 63.5) (xy 147.32 63.5))
     (stroke (width 0) (type default))
@@
     (stroke (width 0) (type default))
   )
+  (wire (pts (xy 129.54 73.66) (xy 129.54 97.79))
+    (stroke (width 0) (type default))
+  )
+  (bus (pts (xy 157.48 109.22) (xy 157.48 110.49))
+    (stroke (width 0) (type default))
+  )
+  (bus (pts (xy 275.59 113.03) (xy 275.59 115.57))
+    (stroke (width 0) (type default))
+  )
   (wire (pts (xy 163.83 46.99) (xy 163.83 49.53))
     (stroke (width 0) (type default))
   )
-  (wire (pts (xy 129.54 73.66) (xy 129.54 97.79))
-    (stroke (width 0) (type default))
-  )
-  (bus (pts (xy 157.48 109.22) (xy 157.48 110.49))
-    (stroke (width 0) (type default))
-  )
-  (bus (pts (xy 275.59 113.03) (xy 275.59 115.57))
-    (stroke (width 0) (type default))
-  )
-  (wire (pts (xy 163.83 53.34) (xy 163.83 49.53))
-    (stroke (width 0) (type default))
-  )
   (wire (pts (xy 168.91 52.07) (xy 168.91 54.61))
     (stroke (width 0) (type default))
   )
-  (wire (pts (xy 172.72 46.99) (xy 168.91 46.99))
-    (stroke (width 0) (type default))
-  )
   (wire (pts (xy 77.47 34.29) (xy 77.47 39.37))
     (stroke (width 0) (type default))
@@
     (stroke (width 0) (type default))
   )
+  (wire (pts (xy 168.91 46.99) (xy 172.72 46.99))
+    (stroke (width 0) (type default))
+  )
   (wire (pts (xy 116.84 100.33) (xy 147.32 100.33))
     (stroke (width 0) (type default))
@@
   )
   (wire (pts (xy 160.02 107.95) (xy 163.83 107.95))
-    (stroke (width 0) (type default))
-  )
-  (wire (pts (xy 172.72 49.53) (xy 163.83 49.53))
     (stroke (width 0) (type default))
   )
@@
     )
   )
-  (symbol (lib_id "Connector:Screw_Terminal_01x03") (at 177.8 49.53 0) (unit 1)
+  (symbol (lib_id "Connector:Screw_Terminal_01x03") (at 177.8 49.53 0) (mirror x) (unit 1)
     (in_bom yes) (on_board yes) (dnp no)
-    (property "Reference" "J2" (at 177.8 58.42 0)
-      (effects (font (size 1.27 1.27)))
-    )
-    (property "Value" "SENSOR" (at 177.8 55.88 0)
+    (property "Reference" "J2" (at 177.8 40.64 0)
+      (effects (font (size 1.27 1.27)))
+    )
+    (property "Value" "SENSOR" (at 177.8 43.18 0)
       (effects (font (size 1.27 1.27)))
     )
@@
   (symbol (lib_id "TM1637__SOP_:TM1637__SOP_") (at 199.39 95.25 0) (mirror y) (unit 1)
     (in_bom yes) (on_board yes) (dnp no)
-    (property "Reference" "IC1" (at 181.61 87.63 0)
+    (property "Reference" "U2" (at 181.61 87.63 0)
       (effects (font (size 1.27 1.27)))
     )
@@
       (project "hardware"
         (path "/4e5cf163-a7ee-4c80-bac0-248feda8733b"
-          (reference "IC1") (unit 1)
+          (reference "U2") (unit 1)
         )
       )
@@
     )
   )
-  (symbol (lib_id "Connector:Screw_Terminal_01x02") (at 45.72 39.37 0) (mirror y) (unit 1)
+  (symbol (lib_id "Connector:Screw_Terminal_01x02") (at 45.72 41.91 180) (unit 1)
     (in_bom yes) (on_board yes) (dnp no)
-    (property "Reference" "J1" (at 45.72 48.26 0)
-      (effects (font (size 1.27 1.27)))
-    )
-    (property "Value" "POWER" (at 45.72 45.72 0)
-      (effects (font (size 1.27 1.27)))
-    )
-    (property "Footprint" "TerminalBlock_Phoenix:TerminalBlock_Phoenix_MPT-0,5-2-2.54_1x02_P2.54mm_Horizontal" (at 45.72 39.37 0)
-      (effects (font (size 1.27 1.27)) hide)
-    )
-    (property "Datasheet" "~" (at 45.72 39.37 0)
-      (effects (font (size 1.27 1.27)) hide)
-    )
+    (property "Reference" "J1" (at 45.72 33.02 0)
+      (effects (font (size 1.27 1.27)))
+    )
+    (property "Value" "POWER" (at 45.72 35.56 0)
+      (effects (font (size 1.27 1.27)))
+    )
+    (property "Footprint" "TerminalBlock_Phoenix:TerminalBlock_Phoenix_MPT-0,5-2-2.54_1x02_P2.54mm_Horizontal" (at 45.72 41.91 0)
+      (effects (font (size 1.27 1.27)) hide)
+    )
+    (property "Datasheet" "~" (at 45.72 41.91 0)
+      (effects (font (size 1.27 1.27)) hide)
+    )
